File: hardware/pcb/openplayer-carrier.kicad_sch (KiCad schematic)
At the start: 15 parts, among them J1 Pi_40pin_IDC, J2 PWR_IN, J3 KEY, J4 BUTTONS, J5 DISPLAY, J6 SWITCH

Commit message: Refactor PCB schematic and build scripts
- Updated the BOM inclusion for test points in the schematic to exclude them from the BOM.
- Modified the build_sch.py script to conditionally set the BOM inclusion based on the reference type.
- Introduced a new build_pcb.py script to automate the generation of the PCB layout from the netlist, including outline, placement, silkscreen, and net definitions.
- Adjusted the placement of components on the PCB to improve layout and accessibility.
- Enhanced text labeling for connectors and pins on the PCB for better clarity and readability.
Parts:
- H1, H2, H3, H4, TP1, TP2, TP3: now left out of the parts list
Changed lines of the file:
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@@
 (label "GND" (at 233.68 54.61 270) (effects (font (size 1.27 1.27)) (justify right bottom)))
 (symbol (lib_id "Connector:TestPoint") (at 213.36 81.28 0) (unit 1)
-(exclude_from_sim no) (in_bom yes) (on_board yes) (dnp no)
+(exclude_from_sim no) (in_bom no) (on_board yes) (dnp no)
 (property "Reference" "TP1" (at 213.36 76.20 0) (effects (font (size 1.27 1.27))))
 (property "Value" "GND" (at 213.36 93.98 0) (effects (font (size 1.27 1.27))))
@@
 (label "GND" (at 213.36 81.28 270) (effects (font (size 1.27 1.27)) (justify right bottom)))
 (symbol (lib_id "Connector:TestPoint") (at 226.06 81.28 0) (unit 1)
-(exclude_from_sim no) (in_bom yes) (on_board yes) (dnp no)
+(exclude_from_sim no) (in_bom no) (on_board yes) (dnp no)
 (property "Reference" "TP2" (at 226.06 76.20 0) (effects (font (size 1.27 1.27))))
 (property "Value" "5V_SYS" (at 226.06 93.98 0) (effects (font (size 1.27 1.27))))
@@
 (label "5V_SYS" (at 226.06 81.28 270) (effects (font (size 1.27 1.27)) (justify right bottom)))
 (symbol (lib_id "Connector:TestPoint") (at 238.76 81.28 0) (unit 1)
-(exclude_from_sim no) (in_bom yes) (on_board yes) (dnp no)
+(exclude_from_sim no) (in_bom no) (on_board yes) (dnp no)
 (property "Reference" "TP3" (at 238.76 76.20 0) (effects (font (size 1.27 1.27))))
 (property "Value" "3V3" (at 238.76 93.98 0) (effects (font (size 1.27 1.27))))
@@
 (label "3V3" (at 238.76 81.28 270) (effects (font (size 1.27 1.27)) (justify right bottom)))
 (symbol (lib_id "Mechanical:MountingHole") (at 213.36 109.22 0) (unit 1)
-(exclude_from_sim no) (in_bom yes) (on_board yes) (dnp no)
+(exclude_from_sim no) (in_bom no) (on_board yes) (dnp no)
 (property "Reference" "H1" (at 213.36 104.14 0) (effects (font (size 1.27 1.27))))
 (property "Value" "M2.5" (at 213.36 121.92 0) (effects (font (size 1.27 1.27))))
@@
 )
 (symbol (lib_id "Mechanical:MountingHole") (at 226.06 109.22 0) (unit 1)
-(exclude_from_sim no) (in_bom yes) (on_board yes) (dnp no)
+(exclude_from_sim no) (in_bom no) (on_board yes) (dnp no)
 (property "Reference" "H2" (at 226.06 104.14 0) (effects (font (size 1.27 1.27))))
 (property "Value" "M2.5" (at 226.06 121.92 0) (effects (font (size 1.27 1.27))))
@@
 )
 (symbol (lib_id "Mechanical:MountingHole") (at 238.76 109.22 0) (unit 1)
-(exclude_from_sim no) (in_bom yes) (on_board yes) (dnp no)
+(exclude_from_sim no) (in_bom no) (on_board yes) (dnp no)
 (property "Reference" "H3" (at 238.76 104.14 0) (effects (font (size 1.27 1.27))))
 (property "Value" "M2.5" (at 238.76 121.92 0) (effects (font (size 1.27 1.27))))
@@
 )
 (symbol (lib_id "Mechanical:MountingHole") (at 251.46 109.22 0) (unit 1)
-(exclude_from_sim no) (in_bom yes) (on_board yes) (dnp no)
+(exclude_from_sim no) (in_bom no) (on_board yes) (dnp no)
 (property "Reference" "H4" (at 251.46 104.14 0) (effects (font (size 1.27 1.27))))
 (property "Value" "M2.5" (at 251.46 121.92 0) (effects (font (size 1.27 1.27))))

Commit message: Update footprint properties for connectors and capacitors in Carrier PCB schematic
Parts:
- C1: value 1000uF 10V -> 470uF 10V; footprint Capacitor_THT:CP_Radial_D10.0mm_P5.00mm -> Capacitor_THT:CP_Radial_D8.0mm_P3.50mm
- J1: footprint Connector_IDC:IDC-Header_2x20_P2.54mm_Vertical -> Connector_IDC:IDC-Header_2x20_P2.54mm_Horizontal
- J2, J3, J6: footprint Connector_JST:JST_XH_B2B-XH-A_1x02_P2.50mm_Vertical -> Connector_JST:JST_XH_S2B-XH-A_1x02_P2.50mm_Horizontal
- J4: footprint Connector_JST:JST_XH_B8B-XH-A_1x08_P2.50mm_Vertical -> Connector_JST:JST_XH_S8B-XH-A_1x08_P2.50mm_Horizontal
- J5: footprint Connector_PinSocket_2.54mm:PinSocket_1x07_P2.54mm_Vertical -> Connector_JST:JST_XH_S7B-XH-A_1x07_P2.50mm_Horizontal
Changed lines of the file:
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@@
 (property "Reference" "J1" (at 101.60 71.12 0) (effects (font (size 1.27 1.27))))
 (property "Value" "Pi_40pin_IDC" (at 101.60 132.08 0) (effects (font (size 1.27 1.27))))
-(property "Footprint" "Connector_IDC:IDC-Header_2x20_P2.54mm_Vertical" (at 101.60 101.60 0) (hide yes) (effects (font (size 1.27 1.27))))
+(property "Footprint" "Connector_IDC:IDC-Header_2x20_P2.54mm_Horizontal" (at 101.60 101.60 0) (hide yes) (effects (font (size 1.27 1.27))))
 (property "Datasheet" "" (at 101.60 101.60 0) (hide yes) (effects (font (size 1.27 1.27))))
 (property "Description" "" (at 101.60 101.60 0) (hide yes) (effects (font (size 1.27 1.27))))
@@
 (property "Reference" "J2" (at 172.72 44.45 0) (effects (font (size 1.27 1.27))))
 (property "Value" "PWR_IN" (at 172.72 46.99 0) (effects (font (size 1.27 1.27))))
-(property "Footprint" "Connector_JST:JST_XH_B2B-XH-A_1x02_P2.50mm_Vertical" (at 172.72 50.80 0) (hide yes) (effects (font (size 1.27 1.27))))
+(property "Footprint" "Connector_JST:JST_XH_S2B-XH-A_1x02_P2.50mm_Horizontal" (at 172.72 50.80 0) (hide yes) (effects (font (size 1.27 1.27))))
 (property "Datasheet" "" (at 172.72 50.80 0) (hide yes) (effects (font (size 1.27 1.27))))
 (property "Description" "" (at 172.72 50.80 0) (hide yes) (effects (font (size 1.27 1.27))))
@@
 (property "Reference" "J3" (at 172.72 74.93 0) (effects (font (size 1.27 1.27))))
 (property "Value" "KEY" (at 172.72 77.47 0) (effects (font (size 1.27 1.27))))
-(property "Footprint" "Connector_JST:JST_XH_B2B-XH-A_1x02_P2.50mm_Vertical" (at 172.72 81.28 0) (hide yes) (effects (font (size 1.27 1.27))))
+(property "Footprint" "Connector_JST:JST_XH_S2B-XH-A_1x02_P2.50mm_Horizontal" (at 172.72 81.28 0) (hide yes) (effects (font (size 1.27 1.27))))
 (property "Datasheet" "" (at 172.72 81.28 0) (hide yes) (effects (font (size 1.27 1.27))))
 (property "Description" "" (at 172.72 81.28 0) (hide yes) (effects (font (size 1.27 1.27))))
@@
 (property "Reference" "J4" (at 172.72 87.63 0) (effects (font (size 1.27 1.27))))
 (property "Value" "BUTTONS" (at 172.72 90.17 0) (effects (font (size 1.27 1.27))))
-(property "Footprint" "Connector_JST:JST_XH_B8B-XH-A_1x08_P2.50mm_Vertical" (at 172.72 101.60 0) (hide yes) (effects (font (size 1.27 1.27))))
+(property "Footprint" "Connector_JST:JST_XH_S8B-XH-A_1x08_P2.50mm_Horizontal" (at 172.72 101.60 0) (hide yes) (effects (font (size 1.27 1.27))))
 (property "Datasheet" "" (at 172.72 101.60 0) (hide yes) (effects (font (size 1.27 1.27))))
 (property "Description" "" (at 172.72 101.60 0) (hide yes) (effects (font (size 1.27 1.27))))
@@
 (property "Reference" "J5" (at 172.72 118.11 0) (effects (font (size 1.27 1.27))))
 (property "Value" "DISPLAY" (at 172.72 120.65 0) (effects (font (size 1.27 1.27))))
-(property "Footprint" "Connector_PinSocket_2.54mm:PinSocket_1x07_P2.54mm_Vertical" (at 172.72 132.08 0) (hide yes) (effects (font (size 1.27 1.27))))
+(property "Footprint" "Connector_JST:JST_XH_S7B-XH-A_1x07_P2.50mm_Horizontal" (at 172.72 132.08 0) (hide yes) (effects (font (size 1.27 1.27))))
 (property "Datasheet" "" (at 172.72 132.08 0) (hide yes) (effects (font (size 1.27 1.27))))
 (property "Description" "" (at 172.72 132.08 0) (hide yes) (effects (font (size 1.27 1.27))))
@@
 (property "Reference" "J6" (at 172.72 59.69 0) (effects (font (size 1.27 1.27))))
 (property "Value" "SWITCH" (at 172.72 62.23 0) (effects (font (size 1.27 1.27))))
-(property "Footprint" "Connector_JST:JST_XH_B2B-XH-A_1x02_P2.50mm_Vertical" (at 172.72 66.04 0) (hide yes) (effects (font (size 1.27 1.27))))
+(property "Footprint" "Connector_JST:JST_XH_S2B-XH-A_1x02_P2.50mm_Horizontal" (at 172.72 66.04 0) (hide yes) (effects (font (size 1.27 1.27))))
 (property "Datasheet" "" (at 172.72 66.04 0) (hide yes) (effects (font (size 1.27 1.27))))
 (property "Description" "" (at 172.72 66.04 0) (hide yes) (effects (font (size 1.27 1.27))))
@@
 (exclude_from_sim no) (in_bom yes) (on_board yes) (dnp no)
 (property "Reference" "C1" (at 213.36 45.72 0) (effects (font (size 1.27 1.27))))
-(property "Value" "1000uF 10V" (at 213.36 63.50 0) (effects (font (size 1.27 1.27))))
-(property "Footprint" "Capacitor_THT:CP_Radial_D10.0mm_P5.00mm" (at 213.36 50.80 0) (hide yes) (effects (font (size 1.27 1.27))))
+(property "Value" "470uF 10V" (at 213.36 63.50 0) (effects (font (size 1.27 1.27))))
+(property "Footprint" "Capacitor_THT:CP_Radial_D8.0mm_P3.50mm" (at 213.36 50.80 0) (hide yes) (effects (font (size 1.27 1.27))))
 (property "Datasheet" "" (at 213.36 50.80 0) (hide yes) (effects (font (size 1.27 1.27))))
 (property "Description" "" (at 213.36 50.80 0) (hide yes) (effects (font (size 1.27 1.27))))

Commit message: Update button and carrier schematics: modify switch positions and add new connector J7
Parts:
- added H5, H6: M2, MountingHole:MountingHole_2.2mm_M2, symbol Mechanical:MountingHole
- added J7: PWR_BTN, Connector_JST:JST_XH_S2B-XH-A_1x02_P2.50mm_Horizontal, symbol Connector_Generic:Conn_01x02
- J1: value Pi_40pin_IDC -> Pi_40pin_socket; footprint Connector_IDC:IDC-Header_2x20_P2.54mm_Horizontal -> Connector_PinSocket_2.54mm:PinSocket_2x20_P2.54mm_Vertical
- J5: footprint Connector_JST:JST_XH_S7B-XH-A_1x07_P2.50mm_Horizontal -> Connector_PinHeader_2.54mm:PinHeader_1x07_P2.54mm_Vertical
Connections:
- net GND: now also J7.2 (Pin_2)
- net PWR_KEY: now also J7.1 (Pin_1)
Changed lines of the file:
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@@
 (exclude_from_sim no) (in_bom yes) (on_board yes) (dnp no)
 (property "Reference" "J1" (at 101.60 71.12 0) (effects (font (size 1.27 1.27))))
-(property "Value" "Pi_40pin_IDC" (at 101.60 132.08 0) (effects (font (size 1.27 1.27))))
-(property "Footprint" "Connector_IDC:IDC-Header_2x20_P2.54mm_Horizontal" (at 101.60 101.60 0) (hide yes) (effects (font (size 1.27 1.27))))
+(property "Value" "Pi_40pin_socket" (at 101.60 132.08 0) (effects (font (size 1.27 1.27))))
+(property "Footprint" "Connector_PinSocket_2.54mm:PinSocket_2x20_P2.54mm_Vertical" (at 101.60 101.60 0) (hide yes) (effects (font (size 1.27 1.27))))
 (property "Datasheet" "" (at 101.60 101.60 0) (hide yes) (effects (font (size 1.27 1.27))))
 (property "Description" "" (at 101.60 101.60 0) (hide yes) (effects (font (size 1.27 1.27))))
@@
 (property "Reference" "J5" (at 172.72 118.11 0) (effects (font (size 1.27 1.27))))
 (property "Value" "DISPLAY" (at 172.72 120.65 0) (effects (font (size 1.27 1.27))))
-(property "Footprint" "Connector_JST:JST_XH_S7B-XH-A_1x07_P2.50mm_Horizontal" (at 172.72 132.08 0) (hide yes) (effects (font (size 1.27 1.27))))
+(property "Footprint" "Connector_PinHeader_2.54mm:PinHeader_1x07_P2.54mm_Vertical" (at 172.72 132.08 0) (hide yes) (effects (font (size 1.27 1.27))))
 (property "Datasheet" "" (at 172.72 132.08 0) (hide yes) (effects (font (size 1.27 1.27))))
 (property "Description" "" (at 172.72 132.08 0) (hide yes) (effects (font (size 1.27 1.27))))
@@
 (label "5V_IN" (at 167.64 66.04 180) (effects (font (size 1.27 1.27)) (justify right bottom)))
 (label "5V_SYS" (at 167.64 68.58 180) (effects (font (size 1.27 1.27)) (justify right bottom)))
+(symbol (lib_id "Connector_Generic:Conn_01x02") (at 172.72 157.48 0) (unit 1)
+(exclude_from_sim no) (in_bom yes) (on_board yes) (dnp no)
+(property "Reference" "J7" (at 172.72 151.13 0) (effects (font (size 1.27 1.27))))
+(property "Value" "PWR_BTN" (at 172.72 153.67 0) (effects (font (size 1.27 1.27))))
+(property "Footprint" "Connector_JST:JST_XH_S2B-XH-A_1x02_P2.50mm_Horizontal" (at 172.72 157.48 0) (hide yes) (effects (font (size 1.27 1.27))))
+(property "Datasheet" "" (at 172.72 157.48 0) (hide yes) (effects (font (size 1.27 1.27))))
+(property "Description" "" (at 172.72 157.48 0) (hide yes) (effects (font (size 1.27 1.27))))
+(pin "1")
+(pin "2")
+(instances (project "openplayer-carrier" (path "/ec122071-abc6-5292-a6b7-15c803da2898" (reference "J7") (unit 1))))
+)
+(label "PWR_KEY" (at 167.64 157.48 180) (effects (font (size 1.27 1.27)) (justify right bottom)))
+(label "GND" (at 167.64 160.02 180) (effects (font (size 1.27 1.27)) (justify right bottom)))
 (symbol (lib_id "Device:C_Polarized") (at 213.36 50.80 0) (unit 1)
 (exclude_from_sim no) (in_bom yes) (on_board yes) (dnp no)
@@
 (instances (project "openplayer-carrier" (path "/ec122071-abc6-5292-a6b7-15c803da2898" (reference "H4") (unit 1))))
 )
+(symbol (lib_id "Mechanical:MountingHole") (at 264.16 109.22 0) (unit 1)
+(exclude_from_sim no) (in_bom no) (on_board yes) (dnp no)
+(property "Reference" "H5" (at 264.16 104.14 0) (effects (font (size 1.27 1.27))))
+(property "Value" "M2" (at 264.16 121.92 0) (effects (font (size 1.27 1.27))))
+(property "Footprint" "MountingHole:MountingHole_2.2mm_M2" (at 264.16 109.22 0) (hide yes) (effects (font (size 1.27 1.27))))
+(property "Datasheet" "" (at 264.16 109.22 0) (hide yes) (effects (font (size 1.27 1.27))))
+(property "Description" "" (at 264.16 109.22 0) (hide yes) (effects (font (size 1.27 1.27))))
+(instances (project "openplayer-carrier" (path "/ec122071-abc6-5292-a6b7-15c803da2898" (reference "H5") (unit 1))))
+)
+(symbol (lib_id "Mechanical:MountingHole") (at 276.86 109.22 0) (unit 1)
+(exclude_from_sim no) (in_bom no) (on_board yes) (dnp no)
+(property "Reference" "H6" (at 276.86 104.14 0) (effects (font (size 1.27 1.27))))
+(property "Value" "M2" (at 276.86 121.92 0) (effects (font (size 1.27 1.27))))
+(property "Footprint" "MountingHole:MountingHole_2.2mm_M2" (at 276.86 109.22 0) (hide yes) (effects (font (size 1.27 1.27))))
+(property "Datasheet" "" (at 276.86 109.22 0) (hide yes) (effects (font (size 1.27 1.27))))
+(property "Description" "" (at 276.86 109.22 0) (hide yes) (effects (font (size 1.27 1.27))))
+(instances (project "openplayer-carrier" (path "/ec122071-abc6-5292-a6b7-15c803da2898" (reference "H6") (unit 1))))
+)
 (sheet_instances (path "/" (page "1")))
