File: hardware/pcb/openplayer-carrier.kicad_sch (KiCad schematic)
At the start: 18 parts, among them J1 Pi_40pin_socket, J2 PWR_IN, J3 KEY, J4 BUTTONS, J5 DISPLAY, J6 SWITCH, J7 PWR_BTN

Commit message: Rev C follow-ups: fix stale requirement lines, drop J5 from the BOM
- docs/pcb-requirements.md §3, §9, §11 no longer mention the ribbon or display cable
- J5 (holes for the display module's own header) excluded from the BOM on
  both the symbol and the footprint, so parity still holds

Co-Authored-By: Claude Opus 5.5 <noreply@anthropic.com>
Claude-Session: https://claude.ai/code/session_0198WPax9Yp1LRqUB5vHM4fv
Parts:
- J5: now left out of the parts list
Changed lines of the file:
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@@
 (label "PWR_KEY" (at 167.64 111.76 180) (effects (font (size 1.27 1.27)) (justify right bottom)))
 (symbol (lib_id "Connector_Generic:Conn_01x07") (at 172.72 132.08 0) (unit 1)
-(exclude_from_sim no) (in_bom yes) (on_board yes) (dnp no)
+(exclude_from_sim no) (in_bom no) (on_board yes) (dnp no)
 (property "Reference" "J5" (at 172.72 118.11 0) (effects (font (size 1.27 1.27))))
 (property "Value" "DISPLAY" (at 172.72 120.65 0) (effects (font (size 1.27 1.27))))
